File: hardware/raccoon_rev2/raccoon_rev2.kicad_sch (KiCad schematic)
At the start: 14 parts, among them J2 AVR-UPDI-6, U2 ATtiny1617-M

Commit message: Added alternate PN as ordered
Parts:
- BT1: ALT PN (none) -> BC-2001
- D1, D2: ALT PN (none) -> MP001247
- R1, R2: ALT PN (none) -> CRCW060310K0FKEA
- R3, R4: ALT PN (none) -> RC0603FR-07330RL
- U2: ALT PN (none) -> ATTINY1617-MN
Changed lines of the file:
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@@
+			)
+		)
+		(property "ALT PN" "RC0603FR-07330RL"
+			(at 185.42 119.38 0)
+			(effects
+				(font
+					(size 1.27 1.27)
+				)
+				(hide yes)
 			)
 		)
@@
 			)
 		)
+		(property "ALT PN" ""
+			(at 77.47 85.09 0)
+			(effects
+				(font
+					(size 1.27 1.27)
+				)
+				(hide yes)
+			)
+		)
 		(pin "1"
 		)
@@
 			)
 		)
+		(property "ALT PN" "ATTINY1617-MN"
+			(at 147.32 96.52 0)
+			(effects
+				(font
+					(size 1.27 1.27)
+				)
+				(hide yes)
+			)
+		)
 		(pin "1"
 		)
@@
 			)
 		)
+		(property "ALT PN" "RC0603FR-07330RL"
+			(at 175.26 119.38 0)
+			(effects
+				(font
+					(size 1.27 1.27)
+				)
+				(hide yes)
+			)
+		)
 		(pin "1"
 		)
@@
 			)
 		)
+		(property "ALT PN" ""
+			(at 210.82 78.74 0)
+			(effects
+				(font
+					(size 1.27 1.27)
+				)
+				(hide yes)
+			)
+		)
 		(pin "5"
 		)
@@
 			)
 		)
+		(property "ALT PN" ""
+			(at 186.69 86.36 90)
+			(effects
+				(font
+					(size 1.27 1.27)
+				)
+				(hide yes)
+			)
+		)
 		(pin "1"
 		)
@@
 		)
 		(property "Manufacturer PN" "0603WAF1002T5E"
+			(at 175.26 86.36 90)
+			(effects
+				(font
+					(size 1.27 1.27)
+				)
+				(hide yes)
+			)
+		)
+		(property "ALT PN" "CRCW060310K0FKEA "
 			(at 175.26 86.36 90)
 			(effects
@@
 			)
 		)
+		(property "ALT PN" "MP001247"
+			(at 175.26 109.22 90)
+			(effects
+				(font
+					(size 1.27 1.27)
+				)
+				(hide yes)
+			)
+		)
 		(pin "1"
 		)
@@
 			)
 		)
+		(property "ALT PN" "MP001247"
+			(at 185.42 109.22 90)
+			(effects
+				(font
+					(size 1.27 1.27)
+				)
+				(hide yes)
+			)
+		)
 		(pin "1"
 		)
@@
 			)
 		)
+		(property "ALT PN" "CRCW060310K0FKEA "
+			(at 175.26 66.04 0)
+			(effects
+				(font
+					(size 1.27 1.27)
+				)
+				(hide yes)
+			)
+		)
 		(pin "1"
 		)
@@
 			)
 		)
+		(property "ALT PN" "BC-2001"
+			(at 68.58 90.17 0)
+			(effects
+				(font
+					(size 1.27 1.27)
+				)
+				(hide yes)
+			)
+		)
 		(pin "1"
 		)
@@
 			)
 		)
+		(property "ALT PN" ""
+			(at 138.43 62.23 0)
+			(effects
+				(font
+					(size 1.27 1.27)
+				)
+				(hide yes)
+			)
+		)
 		(pin "1"
 		)
@@
 			)
 		)
+		(property "ALT PN" ""
+			(at 128.27 62.23 0)
+			(effects
+				(font
+					(size 1.27 1.27)
+				)
+				(hide yes)
+			)
+		)
 		(pin "1"
 		)
@@
 			(at 175.26 92.71 0)
 			(effects
+				(font
+					(size 1.27 1.27)
+				)
+				(hide yes)
+			)
+		)
+		(property "ALT PN" ""
+			(at 175.26 92.71 0)
+			(effects

Commit message: Updated components being placed
Parts:
- C3, R1: now not fitted
Other:
- note added: "Should be a direct pad connection"
Changed lines of the file:
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@@
 		(comment 2 "Current microcontroller choice is definitely overkill")
+	)
+	(text "Should be a direct pad connection"
+		(exclude_from_sim no)
+		(at 182.88 81.28 0)
+		(effects
+			(font
+				(size 1.27 1.27)
+				(italic yes)
+			)
+		)
 	)
 	(text "Jumper to interrupt for current measurement"
@@
 		(in_bom yes)
 		(on_board yes)
-		(dnp no)
+		(dnp yes)
 		(property "Reference" "R1"
 			(at 175.26 83.82 90)
@@
 		(in_bom yes)
 		(on_board yes)
-		(dnp no)
+		(dnp yes)
 		(fields_autoplaced yes)
 		(property "Reference" "C3"
